Commit message: xacro macxro bugfix, change of mounting tf frame, added lens tubes

File: ensenso_description/ensenso.xacro (robot description, xacro)
@@ -4,4 +4,7 @@
   <color rgba="0.1 0.1 1.0 1.0"/>
 </material>
+<material name="Ensenso/Black">
+  <color rgba="0.0 0.0 0.0 1.0"/>
+</material>
   <xacro:macro name="ensenso_N_Series" params="camera parent *origin margin">
     <joint name="${parent}_${camera}_joint" type="fixed">
@@ -12,14 +15,14 @@
     <link name="${camera}_mounting_frame">
       <visual>
-        <origin rpy="1.571 0 3.141" xyz="-0.0875 0.0 -0.0"/>
-        <geometry>
-          <mesh filename="package://ensenso_support/stl_meshes/N30-602-16.stl"/>
-        </geometry>
-        <material name="Ensenso/Blue"/>
-      </visual>
-      <collision>
-        <origin rpy="0 0 0" xyz="-0.01 0.028 0.025"/>
-        <geometry>
-          <box size="${margin+0.20} ${margin+0.056} ${margin+0.05}"/>
+        <origin rpy="0 0 0" xyz="0.00 0.0 0.0"/>
+        <geometry>
+          <mesh filename="package://ensenso_description/stl_meshes/N30-602-16.stl"/>
+        </geometry>
+        <material name="Ensenso/Blue"/>
+      </visual>
+      <collision>
+        <origin rpy="0 0 0" xyz="-0.0085 0.00 0.026"/>
+        <geometry>
+          <box size="${margin+0.192} ${margin+0.050} ${margin+0.052}"/>
         </geometry>
       </collision>
@@ -28,13 +31,13 @@
     <joint name="${camera}_projector_joint" type="fixed">
       <parent link="${camera}_mounting_frame"/>
-      <child link="${camera}_projector_frame"/>
-      <origin xyz="0 0.05 0.026" rpy="-1.570796 0 0"/>
-    </joint>
-    <link name="${camera}_projector_frame"/>
-    <!-- Left lens -->
-    <joint name="${camera}_optical_joint" type="fixed">
-      <parent link="${camera}_mounting_frame"/>
-      <child link="${camera}_left_lens_frame"/>
-      <origin xyz="-0.05 0.05 0.026" rpy="-1.570796 0 0"/>
+      <child link="${camera}_projector_lens_frame"/>
+      <origin xyz="0 0.00 0.05" rpy=" 0 0 0"/>
+    </joint>
+    <link name="${camera}_projector_lens_frame"/>
+    <!-- Left lens -->
+    <joint name="${camera}_left_lense_joint" type="fixed">
+      <parent link="${camera}_mounting_frame"/>
+      <child link="${camera}_left_lens_frame"/>
+      <origin xyz="-0.05 0.00 0.05" rpy=" 0 0 0"/>
     </joint>
     <link name="${camera}_left_lens_frame"/>
@@ -43,24 +46,24 @@
       <parent link="${camera}_mounting_frame"/>
       <child link="${camera}_right_lens_frame"/>
-      <origin xyz="0.05 0.05 0.026" rpy="-1.570796 0 0"/>
+      <origin xyz="0.05 0.00 0.05" rpy=" 0 0 0"/>
     </joint>
     <link name="${camera}_right_lens_frame"/>
   </xacro:macro>
-  <xacro:macro name="ensenso_X200_Series" params="camera parent *origin margin">
-    <joint name="${parent}_${camera}_joint" type="fixed">
-      <xacro:insert_block name="origin"/>
-      <parent link="${parent}" />
-      <child link="${camera}_mounting_frame" />
-    </joint>
-    <link name="${camera}_mounting_frame">
-      <visual>
-        <origin rpy="0 0 0" xyz="0 0 0"/>
-        <geometry>
-          <mesh filename="package://ensenso_support/stl_meshes/X3x-5CP-200.stl"/>
-        </geometry>
-        <material name="Ensenso/Blue"/>
-      </visual>
-      <collision>
-        <origin rpy="0.0 0.0 0.0" xyz="0.0 0.033 0.033"/>
+  <xacro:macro name="ensenso_X200_Series" params="camera parent *origin margin radius_lens_sensor length_lens_sensor radius_lens_projector length_lens_projector">
+    <joint name="${parent}_${camera}_joint" type="fixed">
+      <xacro:insert_block name="origin"/>
+      <parent link="${parent}" />
+      <child link="${camera}_mounting_frame" />
+    </joint>
+    <link name="${camera}_mounting_frame">
+      <visual>
+        <origin rpy="0 0 0" xyz="0 0 0"/>
+        <geometry>
+          <mesh filename="package://ensenso_description/stl_meshes/X3x-5CP-200.stl"/>
+        </geometry>
+        <material name="Ensenso/Blue"/>
+      </visual>
+      <collision>
+        <origin rpy="0.0 0.0 0.0" xyz="0.0 0.0005 0.033"/>
         <geometry>
           <box size="${margin+0.24350} ${margin+0.08} ${margin+0.066}"/>
@@ -68,42 +71,42 @@
       </collision>
     </link>
-    <!-- Projector -->
-    <joint name="${camera}_projector_joint" type="fixed">
-      <parent link="${camera}_mounting_frame"/>
-      <child link="${camera}_projector_frame"/>
-      <origin xyz="0 0.066 0.033" rpy="-1.570796 0 0"/>
-    </joint>
-    <link name="${camera}_projector_frame"/>
-    <!-- Left lens -->
-    <joint name="${camera}_optical_joint" type="fixed">
-      <parent link="${camera}_mounting_frame"/>
-      <child link="${camera}_left_lens_frame"/>
-      <origin xyz="-0.1000 0.066 0.033" rpy="-1.570796 0 0"/>
-    </joint>
-    <link name="${camera}_left_lens_frame"/>
-    <!-- Right lens -->
-    <joint name="${camera}_right_lens_joint" type="fixed">
-      <parent link="${camera}_mounting_frame"/>
-      <child link="${camera}_right_lens_frame"/>
-      <origin xyz="0.1000 0.066 0.033" rpy="-1.570796 0 0"/>
-    </joint>
-    <link name="${camera}_right_lens_frame"/>
-  </xacro:macro>
-  <xacro:macro name="ensenso_X400_Series" params="camera parent *origin margin">
-    <joint name="${parent}_${camera}_joint" type="fixed">
-      <xacro:insert_block name="origin"/>
-      <parent link="${parent}" />
-      <child link="${camera}_mounting_frame" />
-    </joint>
-    <link name="${camera}_mounting_frame">
-      <visual>
-        <origin rpy="0 0 0" xyz="0 0 0"/>
-        <geometry>
-          <mesh filename="package://ensenso_support/stl_meshes/X3x-5CP-400.stl"/>
-        </geometry>
-        <material name="Ensenso/Blue"/>
-      </visual>
-      <collision>
-        <origin rpy="0.0 0.0 0.0" xyz="0.0 0.033 0.033"/>
+    <!-- Left lens -->
+    <joint name="${camera}_left_lens_joint" type="fixed">
+      <parent link="${camera}_mounting_frame"/>
+      <child link="${camera}_left_lens_frame"/>
+      <origin xyz="-0.1067 0.036 0.033" rpy="-1.570796 0 0"/>
+    </joint>
+    <xacro:objective camera="${camera}" margin="${margin}" name="left" radius="${radius_lens_sensor}" length_tube="${length_lens_sensor}"/>
+    <!-- Right lens -->
+    <joint name="${camera}_right_lens_joint" type="fixed">
+      <parent link="${camera}_mounting_frame"/>
+      <child link="${camera}_right_lens_frame"/>
+      <origin xyz="0.1067 0.036 0.033" rpy="-1.570796 0 0"/>
+    </joint>
+    <xacro:objective camera="${camera}" margin="${margin}" name="right" radius="${radius_lens_sensor}" length_tube="${length_lens_sensor}"/>
+    <!-- Projector lens -->
+    <joint name="${camera}_projector_lens_joint" type="fixed">
+      <parent link="${camera}_mounting_frame"/>
+      <child link="${camera}_projector_lens_frame"/>
+      <origin xyz="0 0.04 0.033" rpy="-1.570796 0 0"/>
+    </joint>
+    <xacro:objective camera="${camera}" margin="${margin}" name="projector" radius="${radius_lens_projector}" length_tube="${length_lens_projector}"/>
+  </xacro:macro>
+  <xacro:macro name="ensenso_X400_Series" params="camera parent *origin margin radius_lens_sensor length_lens_sensor radius_lens_projector length_lens_projector">
+    <joint name="${parent}_${camera}_joint" type="fixed">
+      <xacro:insert_block name="origin"/>
+      <parent link="${parent}" />
+      <child link="${camera}_mounting_frame" />
+    </joint>
+    <link name="${camera}_mounting_frame">
+      <visual>
+        <origin rpy="0 0 0" xyz="0 0 0"/>
+        <geometry>
+          <mesh filename="package://ensenso_description/stl_meshes/X3x-5CP-400.stl"/>
+        </geometry>
+        <material name="Ensenso/Blue"/>
+      </visual>
+      <collision>
+        <origin rpy="0.0 0.0 0.0" xyz="0.0 0.0005 0.033"/>
         <geometry>
           <box size="${margin+0.4515} ${margin+0.08} ${margin+0.066}"/>
@@ -111,42 +114,42 @@
       </collision>
     </link>
-    <!-- Projector -->
-    <joint name="${camera}_projector_joint" type="fixed">
-      <parent link="${camera}_mounting_frame"/>
-      <child link="${camera}_projector_frame"/>
-      <origin xyz="0 0.066 0.033" rpy="-1.570796 0 0"/>
-    </joint>
-    <link name="${camera}_projector_frame"/>
-    <!-- Left lens -->
-    <joint name="${camera}_optical_joint" type="fixed">
-      <parent link="${camera}_mounting_frame"/>
-      <child link="${camera}_left_lens_frame"/>
-      <origin xyz="-0.2 0.066 0.033" rpy="-1.570796 0 0"/>
-    </joint>
-    <link name="${camera}_left_lens_frame"/>
-    <!-- Right lens -->
-    <joint name="${camera}_right_lens_joint" type="fixed">
-      <parent link="${camera}_mounting_frame"/>
-      <child link="${camera}_right_lens_frame"/>
-      <origin xyz="0.2 0.066 0.033" rpy="-1.570796 0 0"/>
-    </joint>
-    <link name="${camera}_right_lens_frame"/>
-  </xacro:macro>
-  <xacro:macro name="ensenso_X200_xFA_Series" params="camera parent *origin margin">
-    <joint name="${parent}_${camera}_joint" type="fixed">
-      <xacro:insert_block name="origin"/>
-      <parent link="${parent}" />
-      <child link="${camera}_mounting_frame" />
-    </joint>
-    <link name="${camera}_mounting_frame">
-      <visual>
-        <origin rpy="0 0 0" xyz="0 0 0"/>
-        <geometry>
-          <mesh filename="package://ensenso_support/stl_meshes/X3x-xFA-200.stl"/>
-        </geometry>
-        <material name="Ensenso/Blue"/>
-      </visual>
-      <collision>
-        <origin rpy="0.0 0.0 0.0" xyz="0.0 0.027 0.033"/>
+    <!-- Left lens -->
+    <joint name="${camera}_left_lens_joint" type="fixed">
+      <parent link="${camera}_mounting_frame"/>
+      <child link="${camera}_left_lens_frame"/>
+      <origin xyz="-0.2109 0.036 0.033" rpy="-1.570796 0 0"/>
+    </joint>
+    <xacro:objective camera="${camera}" margin="${margin}" name="left" radius="${radius_lens_sensor}" length_tube="${length_lens_sensor}"/>
+    <!-- Right lens -->
+    <joint name="${camera}_right_lens_joint" type="fixed">
+      <parent link="${camera}_mounting_frame"/>
+      <child link="${camera}_right_lens_frame"/>
+      <origin xyz="0.2109 0.036 0.033" rpy="-1.570796 0 0"/>
+    </joint>
+    <xacro:objective camera="${camera}" margin="${margin}" name="right" radius="${radius_lens_sensor}" length_tube="${length_lens_sensor}"/>
+    <!-- Projector lens -->
+    <joint name="${camera}_projector_lens_joint" type="fixed">
+      <parent link="${camera}_mounting_frame"/>
+      <child link="${camera}_projector_lens_frame"/>
+      <origin xyz="0 0.04 0.033" rpy="-1.570796 0 0"/>
+    </joint>
+    <xacro:objective camera="${camera}" margin="${margin}" name="projector" radius="${radius_lens_projector}" length_tube="${length_lens_projector}"/>
+  </xacro:macro>
+  <xacro:macro name="ensenso_X200_xFA_Series" params="camera parent *origin margin radius_lens_sensor length_lens_sensor radius_lens_projector length_lens_projector">
+    <joint name="${parent}_${camera}_joint" type="fixed">
+      <xacro:insert_block name="origin"/>
+      <parent link="${parent}" />
+      <child link="${camera}_mounting_frame" />
+    </joint>
+    <link name="${camera}_mounting_frame">
+      <visual>
+        <origin rpy="0 0 0" xyz="0 0 0"/>
+        <geometry>
+          <mesh filename="package://ensenso_description/stl_meshes/X3x-xFA-200.stl"/>
+        </geometry>
+        <material name="Ensenso/Blue"/>
+      </visual>
+      <collision>
+        <origin rpy="0.0 0.0 0.0" xyz="0.0 -0.004 0.033"/>
         <geometry>
           <box size="${margin+0.2870} ${margin+0.09} ${margin+0.066}"/>
@@ -154,42 +157,42 @@
       </collision>
     </link>
-    <!-- Projector -->
-    <joint name="${camera}_projector_joint" type="fixed">
-      <parent link="${camera}_mounting_frame"/>
-      <child link="${camera}_projector_frame"/>
-      <origin xyz="0 0.066 0.033" rpy="-1.570796 0 0"/>
-    </joint>
-    <link name="${camera}_projector_frame"/>
-    <!-- Left lens -->
-    <joint name="${camera}_optical_joint" type="fixed">
-      <parent link="${camera}_mounting_frame"/>
-      <child link="${camera}_left_lens_frame"/>
-      <origin xyz="-0.1000 0.066 0.033" rpy="-1.570796 0 0"/>
-    </joint>
-    <link name="${camera}_left_lens_frame"/>
-    <!-- Right lens -->
-    <joint name="${camera}_right_lens_joint" type="fixed">
-      <parent link="${camera}_mounting_frame"/>
-      <child link="${camera}_right_lens_frame"/>
-      <origin xyz="0.1000 0.066 0.033" rpy="-1.570796 0 0"/>
-    </joint>
-    <link name="${camera}_right_lens_frame"/>
-  </xacro:macro>
-  <xacro:macro name="ensenso_X400_xFA_Series" params="camera parent *origin margin">
-    <joint name="${parent}_${camera}_joint" type="fixed">
-      <xacro:insert_block name="origin"/>
-      <parent link="${parent}" />
-      <child link="${camera}_mounting_frame" />
-    </joint>
-    <link name="${camera}_mounting_frame">
-      <visual>
-        <origin rpy="0 0 0" xyz="0 0 0"/>
-        <geometry>
-          <mesh filename="package://ensenso_support/stl_meshes/X3x-xFA-400.stl"/>
-        </geometry>
-        <material name="Ensenso/Blue"/>
-      </visual>
-      <collision>
-        <origin rpy="0.0 0.0 0.0" xyz="0.0 0.027 0.033"/>
+    <!-- Left lens -->
+    <joint name="${camera}_left_lens_joint" type="fixed">
+      <parent link="${camera}_mounting_frame"/>
+      <child link="${camera}_left_lens_frame"/>
+      <origin xyz="-0.117 0.031 0.033" rpy="-1.570796 0 0"/>
+    </joint>
+    <xacro:objective camera="${camera}" margin="${margin}" name="left" radius="${radius_lens_sensor}" length_tube="${length_lens_sensor}"/>
+    <!-- Right lens -->
+    <joint name="${camera}_right_lens_joint" type="fixed">
+      <parent link="${camera}_mounting_frame"/>
+      <child link="${camera}_right_lens_frame"/>
+      <origin xyz="0.117 0.031 0.033" rpy="-1.570796 0 0"/>
+    </joint>
+    <xacro:objective camera="${camera}" margin="${margin}" name="right" radius="${radius_lens_sensor}" length_tube="${length_lens_sensor}"/>
+    <!-- Projector lens -->
+    <joint name="${camera}_projector_lens_joint" type="fixed">
+      <parent link="${camera}_mounting_frame"/>
+      <child link="${camera}_projector_lens_frame"/>
+      <origin xyz="0 0.041 0.033" rpy="-1.570796 0 0"/>
+    </joint>
+    <xacro:objective camera="${camera}" margin="${margin}" name="projector" radius="${radius_lens_projector}" length_tube="${length_lens_projector}"/>
+  </xacro:macro>
+  <xacro:macro name="ensenso_X400_xFA_Series" params="camera parent *origin margin radius_lens_sensor length_lens_sensor radius_lens_projector length_lens_projector">
+    <joint name="${parent}_${camera}_joint" type="fixed">
+      <xacro:insert_block name="origin"/>
+      <parent link="${parent}" />
+      <child link="${camera}_mounting_frame" />
+    </joint>
+    <link name="${camera}_mounting_frame">
+      <visual>
+        <origin rpy="0 0 0" xyz="0 0 0"/>
+        <geometry>
+          <mesh filename="package://ensenso_description/stl_meshes/X3x-xFA-400.stl"/>
+        </geometry>
+        <material name="Ensenso/Blue"/>
+      </visual>
+      <collision>
+        <origin rpy="0.0 0.0 0.0" xyz="0.0 -0.004 0.033"/>
         <geometry>
           <box size="${margin+0.4950} ${margin+0.09} ${margin+0.066}"/>
@@ -197,25 +200,42 @@
       </collision>
     </link>
-    <!-- Projector -->
-    <joint name="${camera}_projector_joint" type="fixed">
-      <parent link="${camera}_mounting_frame"/>
-      <child link="${camera}_projector_frame"/>
-      <origin xyz="0 0.066 0.033" rpy="-1.570796 0 0"/>
-    </joint>
-    <link name="${camera}_projector_frame"/>
-    <!-- Left lens -->
-    <joint name="${camera}_optical_joint" type="fixed">
-      <parent link="${camera}_mounting_frame"/>
-      <child link="${camera}_left_lens_frame"/>
-      <origin xyz="-0.2 0.066 0.033" rpy="-1.570796 0 0"/>
-    </joint>
-    <link name="${camera}_left_lens_frame"/>
-    <!-- Right lens -->
-    <joint name="${camera}_right_lens_joint" type="fixed">
-      <parent link="${camera}_mounting_frame"/>
-      <child link="${camera}_right_lens_frame"/>
-      <origin xyz="0.2 0.066 0.033" rpy="-1.570796 0 0"/>
-    </joint>
-    <link name="${camera}_right_lens_frame"/>
+    <!-- Left lens -->
+    <joint name="${camera}_left_lens_joint" type="fixed">
+      <parent link="${camera}_mounting_frame"/>
+      <child link="${camera}_left_lens_frame"/>
+      <origin xyz="-0.22125 0.031 0.033" rpy="-1.570796 0 0"/>
+    </joint>
+    <xacro:objective camera="${camera}" margin="${margin}" name="left" radius="${radius_lens_sensor}" length_tube="${length_lens_sensor}"/>
+    <!-- Right lens -->
+    <joint name="${camera}_right_lens_joint" type="fixed">
+      <parent link="${camera}_mounting_frame"/>
+      <child link="${camera}_right_lens_frame"/>
+      <origin xyz="0.22125 0.031 0.033" rpy="-1.570796 0 0"/>
+    </joint>
+    <xacro:objective camera="${camera}" margin="${margin}" name="right" radius="${radius_lens_sensor}" length_tube="${length_lens_sensor}"/>
+    <!-- Projector lens -->
+    <joint name="${camera}_projector_lens_joint" type="fixed">
+      <parent link="${camera}_mounting_frame"/>
+      <child link="${camera}_projector_lens_frame"/>
+      <origin xyz="0 0.041 0.033" rpy="-1.570796 0 0"/>
+    </joint>
+    <xacro:objective camera="${camera}" margin="${margin}" name="projector" radius="${radius_lens_projector}" length_tube="${length_lens_projector}"/>
+  </xacro:macro>
+  <xacro:macro name="objective" params="camera margin name radius length_tube">
+    <link name="${camera}_${name}_lens_frame">
+      <visual>
+        <origin xyz="0.0 0.0 ${length_tube / 2.0}" rpy="0 0 0"/>
+        <geometry>
+          <cylinder length="${length_tube}" radius="${radius}"/>
+        </geometry>
+        <material name="Ensenso/Black"/>
+      </visual>
+      <collision>
+        <origin xyz="0.0 0.0 ${(length_tube+2*margin) / 2.0}" rpy="0 0 0"/>
+        <geometry>
+          <cylinder length="${length_tube+2*margin}" radius="${radius+margin}"/>
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
File: ensenso_description/ensenso_N_Series.xacro (robot description, xacro)
@@ -1,10 +1,16 @@
 <?xml version="1.0"?>
 <robot name="ensenso_camera" xmlns:xacro="http://www.ros.org/wiki/xacro">
-  <xacro:include filename="$(find ensenso_support)/ensenso.xacro" />
-  <!-- origin -->
-  <link name="world"/>
-  <xacro:ensenso_N_Series camera="N35" parent="world" margin="0.02">
+  <xacro:include filename="$(find ensenso_description)/ensenso.xacro" />
+  <!-- Parameters -->
+  <!-- Name of the camera -->
+  <xacro:property name="camera" value="N35"/>
+  <!-- Enlarges the bounding box in all directions -->
+  <xacro:property name="margin" value="0.03"/>
+  <!-- Tf Frame, that references to the cameras mounting frame -->
+  <xacro:property name="corresponding_frame_name" value="world"/>
+  <link name="${corresponding_frame_name}"/>
+  <xacro:ensenso_N_Series camera="${camera}" parent="${corresponding_frame_name}" margin="${margin}">
     <origin xyz="0 0 1.0" rpy="0 0 0" />
   </xacro:ensenso_N_Series>
 </robot>
-<!-- example usage with: roslaunch urdf_tutorial display.launch model:=`rospack find ensenso_support`/ensenso_N_Series.xacro gui:=true -->
+<!-- example usage with: roslaunch urdf_tutorial display.launch model:=`rospack find ensenso_description`/ensenso_N_Series.xacro gui:=true -->

File: ensenso_description/ensenso_X200_Series.xacro (robot description, xacro)
@@ -1,10 +1,22 @@
 <?xml version="1.0"?>
 <robot name="ensenso_camera" xmlns:xacro="http://www.ros.org/wiki/xacro">
-  <xacro:include filename="$(find ensenso_support)/ensenso.xacro" />
-  <!-- origin -->
-  <link name="world"/>
-  <xacro:ensenso_X200_Series camera="X200" parent="world" margin="0.02">
+  <xacro:include filename="$(find ensenso_description)/ensenso.xacro" />
+  <!-- Parameters -->
+  <!-- Name of the camera -->
+  <xacro:property name="camera" value="X200"/>
+  <!-- Enlarges the bounding box in all directions -->
+  <xacro:property name="margin" value="0.03"/>
+  <!-- Lens objective properties -->
+  <xacro:property name="lens_length" value="0.05"/>
+  <xacro:property name="lens_radius" value="0.02"/>
+  <!-- Projector objective properties -->
+  <xacro:property name="projector_length" value="0.05"/>
+  <xacro:property name="projector_radius" value="0.02"/>
+  <!-- Tf Frame, that references to the cameras mounting frame -->
+  <xacro:property name="corresponding_frame_name" value="world"/>
+  <link name="${corresponding_frame_name}"/>
+  <xacro:ensenso_X200_Series camera="${camera}" parent="${corresponding_frame_name}" margin="${margin}" radius_lens_sensor="${lens_radius}" length_lens_sensor="${lens_length}" radius_lens_projector="${projector_radius}" length_lens_projector="${projector_length}">
     <origin xyz="0 0 1.0" rpy="0 0 0" />
   </xacro:ensenso_X200_Series>
 </robot>
-<!-- example usage with: roslaunch urdf_tutorial display.launch model:=`rospack find ensenso_support`/ensenso_X200_Series.xacro gui:=true -->
+<!-- example usage with: roslaunch urdf_tutorial display.launch model:=`rospack find ensenso_description`/ensenso_X200_Series.xacro gui:=true -->

File: ensenso_description/ensenso_X200_xFA_Series.xacro (robot description, xacro)
@@ -1,10 +1,22 @@
 <?xml version="1.0"?>
 <robot name="ensenso_camera" xmlns:xacro="http://www.ros.org/wiki/xacro">
-  <xacro:include filename="$(find ensenso_support)/ensenso.xacro" />
-  <!-- origin -->
-  <link name="world"/>
-  <xacro:ensenso_X200_xFA_Series camera="X200_xFA" parent="world" margin="0.02">
+  <xacro:include filename="$(find ensenso_description)/ensenso.xacro" />
+  <!-- Parameters -->
+  <!-- Name of the camera -->
+  <xacro:property name="camera" value="X200_xFA"/>
+  <!-- Enlarges the bounding box in all directions -->
+  <xacro:property name="margin" value="0.03"/>
+  <!-- Lens objective properties -->
+  <xacro:property name="lens_length" value="0.05"/>
+  <xacro:property name="lens_radius" value="0.02"/>
+  <!-- Projector objective properties -->
+  <xacro:property name="projector_length" value="0.05"/>
+  <xacro:property name="projector_radius" value="0.02"/>
+  <!-- Tf Frame, that references to the cameras mounting frame -->
+  <xacro:property name="corresponding_frame_name" value="world"/>
+  <link name="${corresponding_frame_name}"/>
+  <xacro:ensenso_X200_xFA_Series camera="${camera}" parent="${corresponding_frame_name}" margin="${margin}" radius_lens_sensor="${lens_radius}" length_lens_sensor="${lens_length}" radius_lens_projector="${projector_radius}" length_lens_projector="${projector_length}">
     <origin xyz="0 0 1.0" rpy="0 0 0" />
   </xacro:ensenso_X200_xFA_Series>
 </robot>
-<!-- example usage with: roslaunch urdf_tutorial display.launch model:=`rospack find ensenso_support`/ensenso_X200_xFA_Series.xacro gui:=true -->
+<!-- example usage with: roslaunch urdf_tutorial display.launch model:=`rospack find ensenso_description`/ensenso_X200_xFA_Series.xacro gui:=true -->
