Commit message: refactor ensenso.xacro
add N4x / refactor examples

remove projector- and right_lens-links & projector-objective == sensor-objective

remove objectives / integrate Sx / update stl

N_with_xacro.launch should do the job again

File: ensenso_description/ensenso_X400_Series.xacro (robot description, xacro)
@@ -5,25 +5,20 @@
   <!-- Name of the camera -->
   <xacro:arg name="camera" default="X400" />
-  <xacro:property name="camera" value="$(arg camera)" />
+  <xacro:property name="camera_name" value="$(arg camera)" />
   <!-- Enlarges the bounding box in all directions -->
   <xacro:arg name="margin" default="0.03" />
   <xacro:property name="margin" value="$(arg margin)" />
-  <!-- Lens objective properties -->
-  <xacro:arg name="lens_length" default="0.05" />
-  <xacro:property name="lens_length" value="$(arg lens_length)"/>
-  <xacro:arg name="lens_radius" default="0.02" />
-  <xacro:property name="lens_radius" value="$(arg lens_radius)"/>
-  <!-- Projector objective properties -->
-  <xacro:arg name="projector_length" default="0.05" />
-  <xacro:property name="projector_length" value="$(arg projector_length)" />
-  <xacro:arg name="projector_radius" default="0.02" />
-  <xacro:property name="projector_radius" value="$(arg projector_radius)" />
   <!-- Tf Frame, that references to the cameras mounting frame -->
-  <xacro:arg name="corresponding_frame_name" default="world" />
+  <xacro:arg name="corresponding_frame_name" default="base_link" />
   <xacro:property name="corresponding_frame_name" value="$(arg corresponding_frame_name)" />
-  <link name="${corresponding_frame_name}"/>
-  <xacro:ensenso_X400_Series camera="${camera}" parent="${corresponding_frame_name}" margin="${margin}" radius_lens_sensor="${lens_radius}" length_lens_sensor="${lens_length}" radius_lens_projector="${projector_radius}" length_lens_projector="${projector_length}">
-    <origin xyz="0 0 0.0" rpy="0 0 0" />
-  </xacro:ensenso_X400_Series>
+  <xacro:ensenso_X400_Series name="${camera_name}" margin="${margin}"/>
+  <joint name="${corresponding_frame_name}_to_${camera_name}" type="fixed">
+    <parent link="${corresponding_frame_name}" />
+    <child link="${camera_name}" />
+    <origin xyz="0 0 0" rpy="0 0 0" />
+  </joint>
+  <link name="${corresponding_frame_name}" />
 </robot>
-<!-- example usage with: roslaunch urdf_tutorial display.launch model:=`rospack find ensenso_description`/ensenso_X400_Series.xacro gui:=true -->
+<!-- example usage with:
+  roslaunch urdf_tutorial display.launch model:=`rospack find ensenso_description`/ensenso_X400_Series.xacro gui:=true
+-->

Commit message: integrate XQ

File: ensenso_description/ensenso.xacro (robot description, xacro)
@@ -176,3 +176,27 @@
     <link name="${name}_left_lens_frame"/>
   </xacro:macro>
+  <xacro:macro name="ensenso_XQ" params="name margin:=0.03">
+    <link name="${name}">
+      <visual>
+        <origin rpy="0 0 0" xyz="0 0 0"/>
+        <geometry>
+          <mesh filename="package://ensenso_description/stl_meshes/X3x-Q.stl"/>
+        </geometry>
+        <material name="Ensenso/Blue"/>
+      </visual>
+      <collision>
+        <origin rpy="0.0 0.0 0.0" xyz="0.0 0.0 ${margin/2 + 0.11}"/>
+        <geometry>
+          <box size="${margin+0.650} ${margin+0.616} ${margin+0.22}"/>
+        </geometry>
+      </collision>
+    </link>
+    <!-- Left lens -->
+    <joint name="${name}_left_lens_joint" type="fixed">
+      <parent link="${name}"/>
+      <child link="${name}_left_lens_frame"/>
+      <origin xyz="-0.22125 0 0.063" rpy="0 0 0"/>
+    </joint>
+    <link name="${name}_left_lens_frame"/>
+  </xacro:macro>
 </robot>

Commit message: ensenso_description: Add support for C-Series

File: ensenso_description/ensenso.xacro (robot description, xacro)
@@ -7,4 +7,7 @@
   <color rgba="0.0 0.0 0.0 1.0"/>
 </material>
+<material name="Ensenso/DarkGrey">
+  <color rgba="0.35 0.35 0.35 1.0"/>
+</material>
 <xacro:macro name="ensenso_Sx_Series" params="name margin:=0.03">
     <link name="${name}">
@@ -176,3 +179,51 @@
     <link name="${name}_left_lens_frame"/>
   </xacro:macro>
+  <xacro:macro name="ensenso_CxS_Series" params="name margin:=0.03">
+    <link name="${name}">
+      <visual>
+        <origin rpy="0 0 0" xyz="0 0 0"/>
+        <geometry>
+          <mesh filename="package://ensenso_description/stl_meshes/Cx-S.stl"/>
+        </geometry>
+        <material name="Ensenso/DarkGrey"/>
+      </visual>
+      <collision>
+        <origin rpy="0.0 0.0 0.0" xyz="0.0 0.0 ${0.10/2}"/>
+        <geometry>
+          <box size="${margin+0.300} ${margin+0.06} ${margin+0.10+0.02}"/>
+        </geometry>
+      </collision>
+    </link>
+    <!-- Left lens -->
+    <joint name="${name}_left_lens_joint" type="fixed">
+      <parent link="${name}"/>
+      <child link="${name}_left_lens_frame"/>
+      <origin xyz="-0.123 0.0 0.063" rpy="0 0 0"/>
+    </joint>
+    <link name="${name}_left_lens_frame"/>
+  </xacro:macro>
+  <xacro:macro name="ensenso_CxM_Series" params="name margin:=0.03">
+    <link name="${name}">
+      <visual>
+        <origin rpy="0 0 0" xyz="0 0 0"/>
+        <geometry>
+          <mesh filename="package://ensenso_description/stl_meshes/Cx-M.stl"/>
+        </geometry>
+        <material name="Ensenso/DarkGrey"/>
+      </visual>
+      <collision>
+        <origin rpy="0.0 0.0 0.0" xyz="0.0 0.0 ${0.10/2}"/>
+        <geometry>
+          <box size="${margin+0.510} ${margin+0.06} ${margin+0.10+0.02}"/>
+        </geometry>
+      </collision>
+    </link>
+    <!-- Left lens -->
+    <joint name="${name}_left_lens_joint" type="fixed">
+      <parent link="${name}"/>
+      <child link="${name}_left_lens_frame"/>
+      <origin xyz="-0.22125 0 0.063" rpy="0 0 0"/>
+    </joint>
+    <link name="${name}_left_lens_frame"/>
+  </xacro:macro>
 </robot>

Commit message: ensenso_description: Fix C-Series X and Z offset

File: ensenso_description/ensenso.xacro (robot description, xacro)
@@ -199,5 +199,5 @@
       <parent link="${name}"/>
       <child link="${name}_left_lens_frame"/>
-      <origin xyz="-0.123 0.0 0.063" rpy="0 0 0"/>
+      <origin xyz="${-0.240/2} 0.0 0.032" rpy="0 0 0"/>
     </joint>
     <link name="${name}_left_lens_frame"/>
@@ -223,5 +223,5 @@
       <parent link="${name}"/>
       <child link="${name}_left_lens_frame"/>
-      <origin xyz="-0.22125 0 0.063" rpy="0 0 0"/>
+      <origin xyz="${-0.455/2} 0 0.032" rpy="0 0 0"/>
     </joint>
     <link name="${name}_left_lens_frame"/>

Commit message: ensenso_description: Add support for Cx-L

File: ensenso_description/ensenso.xacro (robot description, xacro)
@@ -227,3 +227,27 @@
     <link name="${name}_left_lens_frame"/>
   </xacro:macro>
+  <xacro:macro name="ensenso_CxL_Series" params="name margin:=0.03">
+    <link name="${name}">
+      <visual>
+        <origin rpy="0 0 ${pi}" xyz="0 0 0"/>
+        <geometry>
+          <mesh filename="package://ensenso_description/stl_meshes/Cx-L.stl"/>
+        </geometry>
+        <material name="Ensenso/DarkGrey"/>
+      </visual>
+      <collision>
+        <origin rpy="0.0 0.0 0.0" xyz="0.0 0.0 ${0.10/2}"/>
+        <geometry>
+          <box size="${margin+0.910} ${margin+0.06} ${margin+0.10+0.02}"/>
+        </geometry>
+      </collision>
+    </link>
+    <!-- Left lens -->
+    <joint name="${name}_left_lens_joint" type="fixed">
+      <parent link="${name}"/>
+      <child link="${name}_left_lens_frame"/>
+      <origin xyz="${-0.850/2} 0 0.032" rpy="0 0 0"/>
+    </joint>
+    <link name="${name}_left_lens_frame"/>
+  </xacro:macro>
 </robot>

Commit message: ensenso_description: Add support for B-Series

File: ensenso_description/ensenso.xacro (robot description, xacro)
@@ -251,3 +251,27 @@
     <link name="${name}_left_lens_frame"/>
   </xacro:macro>
+  <xacro:macro name="ensenso_Bx_Series" params="name margin:=0.03">
+    <link name="${name}">
+      <visual>
+        <origin rpy="0 0 ${pi}" xyz="0 0 0"/>
+        <geometry>
+          <mesh filename="package://ensenso_description/stl_meshes/Bx.stl"/>
+        </geometry>
+        <material name="Ensenso/DarkGrey"/>
+      </visual>
+      <collision>
+        <origin rpy="0.0 0.0 0.0" xyz="0.0 0.0 ${(0.104+0.01)/2}"/>
+        <geometry>
+          <box size="${margin+0.120} ${margin+0.056} ${margin+0.104+0.02}"/>
+        </geometry>
+      </collision>
+    </link>
+    <!-- Left lens -->
+    <joint name="${name}_left_lens_joint" type="fixed">
+      <parent link="${name}"/>
+      <child link="${name}_left_lens_frame"/>
+      <origin xyz="${-0.075/2} 0 0.090" rpy="0 0 0"/>
+    </joint>
+    <link name="${name}_left_lens_frame"/>
+  </xacro:macro>
 </robot>
